File: vw-gti-12v-distribution.kicad_sch (KiCad schematic)
At the start: 4 parts, among them J1 IN_12V, J2 OUT_DASHCAM, J3 OUT_PHONE, J4 OUT_BOOST

Commit message: Switch to SMD PicoSpoX and add ACC + extra outputs
Parts:
- removed J3: OUT_PHONE, PicoSpoX:PicoSpoX_1x02_P3.00mm_THT, symbol Connector_Generic:Conn_01x02
- removed J4: OUT_BOOST, PicoSpoX:PicoSpoX_1x02_P3.00mm_THT, symbol Connector_Generic:Conn_01x02
- added J3: OUT_DASHCAM, PicoSpoX:PicoSpoX_1x03_P3.00mm_SMD, symbol Connector_Generic:Conn_01x03
- added J4: OUT_PHONE, PicoSpoX:PicoSpoX_1x03_P3.00mm_SMD, symbol Connector_Generic:Conn_01x03
- added J5: OUT_BOOST, PicoSpoX:PicoSpoX_1x03_P3.00mm_SMD, symbol Connector_Generic:Conn_01x03
- added J6: OUT_SPARE1, PicoSpoX:PicoSpoX_1x03_P3.00mm_SMD, symbol Connector_Generic:Conn_01x03
- added J7: OUT_SPARE2, PicoSpoX:PicoSpoX_1x03_P3.00mm_SMD, symbol Connector_Generic:Conn_01x03
- J1: value IN_12V -> IN_BATT; footprint PicoSpoX:PicoSpoX_1x02_P3.00mm_THT -> PicoSpoX:PicoSpoX_1x02_P3.00mm_SMD
- J2: value OUT_DASHCAM -> IN_ACC; footprint PicoSpoX:PicoSpoX_1x02_P3.00mm_THT -> PicoSpoX:PicoSpoX_1x02_P3.00mm_SMD
Other:
- note added: "+12V_ACC"
- note added: "+12V_BATT"
- note removed: "+12V"
