File: car-12v-power-distribution-pcb.kicad_sch (KiCad schematic)
At the start: 7 parts, among them J1 IN_BATT, J2 IN_ACC, J3 OUT_DASHCAM, J4 OUT_PHONE, J5 OUT_BOOST, J6 OUT_SPARE1, J7 OUT_SPARE2

Commit message: Rename project to car-12v-power-distribution-pcb
Other:
- title: VW GTI 12V Distribution -> Car 12V Power Distribution
Changed lines of the file:
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@@
   (paper "A4")
   (title_block
-    (title "VW GTI 12V Distribution")
+    (title "Car 12V Power Distribution")
     (date "2026-02-28")
     (rev "B")
